Commit message: Poprawiony urdf, zmienione jointy, dodany joint bazowy
Joint 3 nieruchomy, joint2 ruchomy

File: lab02/urdf/movingjoints.xacro (robot description, xacro)
@@ -23,4 +23,6 @@
 <xacro:property name="z3" value="1"/>
 <xacro:property name="l3" value="1"/>
+	<link name="base_link1">
+	</link>
 	<link name="base_link">
 		<visual>
@@ -56,5 +58,5 @@
 		<visual>
 			<geometry>
-				<cylinder length="0.4" radius="0.3"/>
+				<box size=".1 .2 .3"/>
 			</geometry>
 			<material name="white">
@@ -63,4 +65,10 @@
 		</visual>
 	</link>
+	<joint name="joint" type="revolute">
+		<parent link="base_link1"/>
+		<child link="base_link"/>
+		<limit effort="1000.0" lower="-3.5" upper="1.6" velocity="0.5"/>
+		<axis xyz="0 0 1" />
+	</joint>
 	<joint name="joint1" type="revolute">
 		<parent link="base_link"/>
@@ -70,15 +78,16 @@
 		<axis xyz="0 0 1" />
 	</joint>
-	<joint name="joint2" type="revolute">
+	<joint name="joint2" type="prismatic">
 		<parent link="link1"/>
 		<child link="link2"/>
 		<origin xyz="${x2} ${y2} ${z2}" rpy="${r2} ${p2} ${yy2}" />
-		<limit effort="1000.0" lower="-0.93" upper="4" velocity="0.5"/>
-		<axis xyz="0 1 0" />
+		<limit effort="1000.0" lower="-0.81" upper="-0.05" velocity="0.5"/>
+		<axis xyz="0 0 1" />
 	</joint>
-	<joint name="joint3" type="continuous">
+	<joint name="joint3" type="fixed">
 		<parent link="link2"/>
 		<child link="link3"/>
 		<origin xyz="${x3} ${y3} ${z3}" rpy="${r3} ${p3} ${yy3}" />
+		<limit effort="1000.0" lower="-0.6" upper="-0.11" velocity="0.5"/>
 		<axis xyz="0 0 1" />
 	</joint>
