Commit message: Ostateczna wersja lab3

File: anrobot_description/urdf/movable.urdf (robot description, URDF)
Before this commit: robot test_robot, 7 links, 6 joints
Links:
- link arm1: geometry visual cylinder length=2 radius=0.15
- link arm2: geometry visual cylinder length=1 radius=0.1
- link arm3: geometry visual box size=.07 .07 2
- link base_link: geometry visual cylinder length=0.6 radius=0.15
- link link1: geometry visual box size=.1 .1 .1
- link link2: geometry visual box size=.1 .1 .1
- link link3: geometry visual box size=.1 .2 .3
Joints:
- joint joint3: limit lower=0.3 upper=3 effort=1000.0 velocity=0.5 -> lower=0.5 upper=2 effort=1000.0 velocity=0.5
